File: PresToe_BMS_48V.kicad_pcb (KiCad board)
At the start: 2 copper layers, 0 parts

Commit message: Basic footprint layout added
Parts:
- added C1: 2.7nF, Capacitor_SMD:C_0603_1608Metric, F.Cu at (76.5, 73.5)
- added C2: 1uF, Capacitor_SMD:C_0603_1608Metric, F.Cu at (51.5, 36.9)
- added C3: 22uF, Capacitor_SMD:C_0603_1608Metric, F.Cu at (51.5, 29.4)
- added C4: 3.3nF, Capacitor_SMD:C_0603_1608Metric, F.Cu at (46.8, 73.5)
- added C5: 470nF, Capacitor_SMD:C_0603_1608Metric, F.Cu at (78.3, 73.5)
- added D1: GREEN, LED_SMD:LED_0603_1608Metric, F.Cu at (92.8, 28.8)
- added D2: GREEN, LED_SMD:LED_0603_1608Metric, F.Cu at (92.8, 31.5)
- added D3: RED, LED_SMD:LED_0603_1608Metric, F.Cu at (92.8, 34.2)
- added J1: XT90PB-F, xt90:XT90PBF, F.Cu at (38.5, 61.2)
- added J2: XT90PB-F, xt90:XT90PBF, F.Cu at (87.0, 61.2)
- added J3: XT30PW-M, XT30PW-M:AMASS_XT30PW-M, F.Cu at (35.3, 46.5)
- added J4: S3B-XH-A, S3B_XH_A:JST_S3B-XH-A, F.Cu at (36.0, 33.2)
- added J5: Conn_01x06_Pin, Connector_JST:JST_EH_S6B-EH_1x06_P2.50mm_Horizontal, F.Cu at (87.0, 39.0)
- added P1: T93YA203JT20, 20k_potentiometer:POT_T93YA_VIS, F.Cu at (71.2, 78.2)
- added Q1: IAUS200N08S5N023ATMA1, IAUS200N08S5N023ATMA1:TRANS_IAUS200N08S5N023ATMA1, F.Cu at (51.2, 62.0)
- added Q2: IAUS200N08S5N023ATMA1, IAUS200N08S5N023ATMA1:TRANS_IAUS200N08S5N023ATMA1, F.Cu at (63.0, 62.0)
- added Q3: IAUS200N08S5N023ATMA1, IAUS200N08S5N023ATMA1:TRANS_IAUS200N08S5N023ATMA1, F.Cu at (74.5, 62.0)
- added R1: 100k, Resistor_SMD:R_0603_1608Metric, F.Cu at (67.8, 73.5)
- added R10: 150, Resistor_SMD:R_0603_1608Metric, F.Cu at (87.3, 31.5)
- added R11: 150, Resistor_SMD:R_0603_1608Metric, F.Cu at (87.3, 34.5)
- added R12: 51k, Resistor_SMD:R_0603_1608Metric, F.Cu at (57.5, 34.8)
- added R13: 5k, Resistor_SMD:R_0603_1608Metric, F.Cu at (59.5, 34.8)
- added R14: 100k, Resistor_SMD:R_0603_1608Metric, F.Cu at (53.8, 73.5)
- added R15: 1.6k, Resistor_SMD:R_0603_1608Metric, F.Cu at (56.5, 73.5)
- added R2: 10, Resistor_SMD:R_0603_1608Metric, F.Cu at (69.5, 73.5)
- added R3: 2.2, Resistor_SMD:R_0603_1608Metric, F.Cu at (71.3, 73.5)
- added R4: 2.2, Resistor_SMD:R_0603_1608Metric, F.Cu at (73.0, 73.5)
- added R5: 2.2, Resistor_SMD:R_0603_1608Metric, F.Cu at (74.8, 73.5)
- added R6: 470k, Resistor_SMD:R_0603_1608Metric, F.Cu at (48.5, 73.5)
- added R7: 3.4k, Resistor_SMD:R_0603_1608Metric, F.Cu at (50.3, 73.5)
- added R8: 11k, Resistor_SMD:R_0603_1608Metric, F.Cu at (52.0, 73.5)
- added R9: 150, Resistor_SMD:R_0603_1608Metric, F.Cu at (87.3, 28.8)
- added R_FBB1: 32.4k, Resistor_SMD:R_0603_1608Metric, F.Cu at (48.8, 36.1)
- added R_FBT1: 100k, Resistor_SMD:R_0603_1608Metric, F.Cu at (54.3, 36.0)
- added R_SNS1: 300u, Resistor_SMD:Custom_R_300u, F.Cu at (75.5, 47.0)
- added R_SNS2: 300u, Resistor_SMD:Custom_R_300u, F.Cu at (57.0, 47.0)
- added SW1: DS04-254-1-01BK-SMT, dip_1:SW_DS04-254_CUD, F.Cu at (51.8, 78.0)
- added TP1: TestPoint, TestPoint:TestPoint_Pad_D2.0mm, F.Cu at (64.3, 79.5)
- added TP2: TestPoint, TestPoint:TestPoint_Pad_D2.0mm, F.Cu at (60.8, 79.5)
- added U1: PTPS48000QDGXRQ1, tps4800:VSSOP19-DGX_TEX, F.Cu at (62.5, 74.5)
- added U2: TPSM265R1SILR, TPSM265R1SILR:MODULE_TPSM265R1SILR, F.Cu at (51.5, 33.6)
- added U3: INA241A2QDGKRQ1, ul_INA241A1QDGKRQ1:VSSOP8_DGK_TEX, F.Cu at (66.3, 37.0)
- added U4: TLV9051IDBVR, TLV9051IDBVR:SOT23_DBV_TEX, F.Cu at (58.5, 30.1)
- added U5: MCP3202T-CI/MS, MCP3202:SOIC8-N_MC_MCH, F.Cu at (66.1, 31.1)
- added U6: ISO6741DWR, ISO6741DWR:SOIC127P1030X265-16N, F.Cu at (77.5, 33.5)
