File: PresToe_BMS_48V.kicad_pcb (KiCad board)
At the start: 2 copper layers, 45 parts, among them J1 XT90PB-F, J2 XT90PB-F, J3 XT30PW-M, J4 S3B-XH-A, J5 Conn_01x06_Pin, P1 T93YA203JT20, Q1 IAUS200N08S5N023ATMA1, Q2 IAUS200N08S5N023ATMA1, Q3 IAUS200N08S5N023ATMA1, SW1 DS04-254-1-01BK-SMT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

Commit message: finalized, remaining final checks
Parts:
- added H1: MountingHole, MountingHole:MountingHole_3.2mm_M3_Pad_Via, F.Cu at (34.2, 32.0)
- added H2: MountingHole, MountingHole:MountingHole_3.2mm_M3_Pad_Via, F.Cu at (93.0, 32.0)
- added H3: MountingHole, MountingHole:MountingHole_3.2mm_M3_Pad_Via, F.Cu at (34.2, 78.2)
- added H4: MountingHole, MountingHole:MountingHole_3.2mm_M3_Pad_Via, F.Cu at (93.0, 78.2)
- moved D3 52.6 mm to (40.3, 37.4)
- moved D2 52.5 mm to (40.3, 33.6)
- moved D1 52.5 mm to (40.3, 29.5)
- moved R11 43.4 mm to (44.0, 37.4)
- moved R10 43.3 mm to (44.0, 33.6)
- moved R9 43.3 mm to (44.0, 29.5)
- moved P1 39.1 mm to (38.2, 57.3), turned to -90 degrees
- moved TP1 33.6 mm to (32.0, 70.4)
- moved J4 29.2 mm to (65.1, 29.9), turned to 180 degrees
- moved C1 28.8 mm to (52.9, 57.1)
- moved C5 28.8 mm to (54.7, 57.1), turned to 90 degrees
- moved R1 28.8 mm to (44.1, 57.1)
- moved R2 28.8 mm to (45.9, 57.1)
- moved R3 28.8 mm to (47.6, 57.1)
- moved R4 28.8 mm to (49.4, 57.1)
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Connections:
- U4 pad 1: Net-(U4-OUT) -> Net-(U4--IN)
- U4 pad 4: V_ADC -> Net-(U4--IN)
- U5 pad 3: Net-(U4-OUT) -> Net-(U4--IN)
Routing:
- net V_out: track 0.00 -> 120.1 mm, vias 0 -> 654
- net SPI_VIN: track 0.00 -> 102.8 mm, vias 0 -> 2
- net V_load: track 0.00 -> 96.9 mm, vias 0 -> 427
- net 5V: track 0.00 -> 90.8 mm
- net SPI_GND: track 0.00 -> 87.7 mm, vias 0 -> 1
- net SPI_MISO: track 0.00 -> 81.3 mm, vias 0 -> 1
- net INP: track 0.00 -> 80.0 mm, vias 0 -> 1
- net SPI_MOSI: track 0.00 -> 78.7 mm, vias 0 -> 2
- net SPI_SCLK: track 0.00 -> 66.9 mm, vias 0 -> 1
- net SPI_*CS: track 0.00 -> 64.3 mm, vias 0 -> 1
- net V_in: track 0.00 -> 61.5 mm, vias 0 -> 532
- net GND: track 0.00 -> 61.3 mm, vias 0 -> 20
- net Net-(U1-TMR): track 0.00 -> 41.4 mm, vias 0 -> 2
- net FLT_GD: track 0.00 -> 40.3 mm
- net Net-(U1-PD): track 0.00 -> 37.6 mm, vias 0 -> 2
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- added copper zone on In1.Cu, net GND
- added copper zone on B.Cu, net V_in
- added copper zone on F.Cu, net V_in
- added copper zone on In2.Cu, net V_in
- added copper zone on In3.Cu, net V_in
- added copper zone on In4.Cu, net V_in
- added copper zone on B.Cu, net V_load
- added copper zone on F.Cu, net V_load
- added copper zone on In2.Cu, net V_load
- added copper zone on In3.Cu, net V_load
- added copper zone on In4.Cu, net V_load
- added copper zone on B.Cu, net V_out
- added copper zone on F.Cu, net V_out
- added copper zone on In2.Cu, net V_out
- added copper zone on In3.Cu, net V_out
- added copper zone on In4.Cu, net V_out
Other:
- board outline added: 70.2 x 58.2 mm
- copper layers 2 -> 6
- board text added: "*"
- board text added: "*CS SCLK MOSI MISO MCU_VIN MCU_GND"
- board text added: "+"
- board text added: "-"
- board text added: "FLT"
- board text added: "GATE"
- board text added: "PWR"
- board text added: "PresToe Robot 48V DC BMS DARoS Lab Aryaman Ghura"
- board text added: "V_IN"
- board text added: "V_OUT"

Commit message: fixed bugs, finalized design
Parts:
- removed the H3 at (34.2, 78.2)
- added C10: 0.1uF, Capacitor_SMD:C_0603_1608Metric, F.Cu at (52.2, 40.7)
- added C11: 0.1uF, Capacitor_SMD:C_0603_1608Metric, F.Cu at (49.1, 40.7)
- added C6: 0.1uF, Capacitor_SMD:C_0603_1608Metric, F.Cu at (51.2, 57.1)
- added C7: 0.1uF, Capacitor_SMD:C_0603_1608Metric, F.Cu at (87.8, 27.5)
- added C8: 0.1uF, Capacitor_SMD:C_0603_1608Metric, F.Cu at (79.6, 27.6)
- added C9: 0.1uF, Capacitor_SMD:C_0603_1608Metric, F.Cu at (83.8, 27.6)
- added NT1: NetTie_2, NetTie:NetTie-2_SMD_Pad2.0mm, F.Cu at (37.9, 76.8)
- P1: footprint 20k_potentiometer:POT_T93YA_VIS -> 89PR20KLF:RES3_89P_TTE
- moved P1 21.6 mm to (34.0, 78.5), turned to 90 degrees
- moved R13 17.8 mm to (90.7, 41.3), turned to 180 degrees
- moved R12 17.0 mm to (90.7, 43.3), turned to 0 degrees
- moved TP2 14.4 mm to (37.8, 56.2)
- moved TP1 14.3 mm to (32.7, 56.2)
- moved SW1 4.27 mm to (39.3, 66.0), turned to -90 degrees
- moved R1 1.60 mm to (42.5, 57.1)
- moved R2 1.60 mm to (44.3, 57.1)
- moved R3 1.60 mm to (46.0, 57.1)
- moved R4 1.60 mm to (47.8, 57.1)
- moved R5 1.60 mm to (49.5, 57.1)
- renumbered H4 to H3
Connections:
- J1 pad 1: GND -> PWR_GND
- J2 pad 1: GND -> PWR_GND
- U6 pad 11: Net-(U5-DIN) -> Net-(U5-DOUT)
- U6 pad 14: Net-(U5-DOUT) -> Net-(U5-DIN)
Routing:
- net GND: track 61.3 -> 9.91 mm, vias 20 -> 35
- net 5V: track 90.8 -> 119.1 mm
- net Net-(U1-TMR): track 41.4 -> 22.1 mm, vias 2 -> 0
- net Net-(U4-+IN): track 12.6 -> 30.5 mm
- net Net-(P1-Pad2): track 28.8 -> 16.1 mm
- net Net-(U5-DIN): track 32.1 -> 23.3 mm
- net Net-(U5-DOUT): track 20.1 -> 26.9 mm
- net Net-(U1-ISCP): track 26.6 -> 32.4 mm, vias 0 -> 2
- net Net-(U3-OUT): track 16.6 -> 11.4 mm
- net SPI_VIN: track 102.8 -> 107.4 mm
- net V_in: track 61.5 -> 65.4 mm, vias 532 -> 508
- net Net-(Q3-Pad1): track 26.1 -> 29.8 mm
- net Net-(Q2-Pad1): track 26.4 -> 29.1 mm
- net V_load: track 96.9 -> 94.2 mm
- net Net-(Q1-Pad1): track 32.5 -> 34.1 mm
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- added copper zone on In2.Cu, net GND
- added copper zone on In1.Cu, net PWR_GND
- removed copper zone on In1.Cu, net GND
Other:
- board text added: "CH0: Current Precision: ±0.41A Range: [-833A, 833A] CH1: Voltage Precision: ±14mV Range: [0V, 56V]"
- board text added: "ESTOP"
- board text added: "MOSFET1"
- board text added: "MOSFET2"
- board text added: "MOSFET3"
- board text added: "R = R_iscp = R_TP1 - R_TP2 I_sc = (R*2e-6+19e-3)/(150e-6) I_sc_min ≈ 148A; R_min ≈ 1.6kΩ I_sc_max ≈ 415A; R_max ≈ 21.6kΩ ΔI_sc/Rev ≈ 13.3A"
- board text added: "R_ISCP"
- board text added: "SPI"
- board text added: "Switch"
- board text added: "UV = 42.5 ± 0.84 V OV = 54.6 ± 1.09 V T_sc (RST) = 45.3us T_sc (STP) = 48us - RST attempts to reopen GATE after SC detected - STP powers off GATE and requires hard restart"
- board text added: "↻"

Commit message: Finalized V1
Parts:
- added G***: LOGO, LOGO, F.Cu at (96.3, 65.2)
- added G***: LOGO, LOGO, F.Cu at (91.2, 65.8)
- C2: footprint Capacitor_SMD:C_0603_1608Metric -> Capacitor_SMD:C_0805_2012Metric
- C3: footprint Capacitor_SMD:C_0603_1608Metric -> Capacitor_SMD:C_1210_3225Metric
- moved C10 2.81 mm to (54.7, 39.3)
- moved C11 2.23 mm to (50.9, 39.3)
- moved C3 0.84 mm to (54.8, 46.1)
- moved C2 0.28 mm to (47.3, 46.3)
Routing:
- net SPI_VIN: track 107.4 -> 104.9 mm
- net 5V: track 119.1 -> 116.9 mm
- net ESTOP: track 26.3 -> 25.6 mm
Other:
- board text added: "- RST attempts to reopen GATE after SC detected - STP powers off GATE and requires hard restart"
- board text added: "CH0: Current Precision: ±0.41A Range: [-833.3A, 833.3A]"
- board text added: "CH1: Voltage Precision: ±14mV Range: [0V, 56V]"
- board text added: "PresToe Robot 48V DC BMS V1 DARoS Lab Aryaman Ghura"
- board text added: "R = R_iscp = R_TP1 - R_TP2 I_sc = (R*2e-6+19e-3)/(150e-6) I_sc_min ≈ 148A; R_min ≈ 1.6kΩ I_sc_max ≈ 415A; R_max ≈ 21.6kΩ ΔI_sc/Rev ≈ 13.3A; ΔR/Rev = 1kΩ"
- board text added: "T_sc (RST) = 45.3us T_sc (STP) = 48us"
- board text added: "UV = 42.5 ± 0.84 V OV = 54.6 ± 1.09 V"
- board text removed: "CH0: Current Precision: ±0.41A Range: [-833A, 833A] CH1: Voltage Precision: ±14mV Range: [0V, 56V]"
- board text removed: "PresToe Robot 48V DC BMS DARoS Lab Aryaman Ghura"
- board text removed: "R = R_iscp = R_TP1 - R_TP2 I_sc = (R*2e-6+19e-3)/(150e-6) I_sc_min ≈ 148A; R_min ≈ 1.6kΩ I_sc_max ≈ 415A; R_max ≈ 21.6kΩ ΔI_sc/Rev ≈ 13.3A"
- board text removed: "UV = 42.5 ± 0.84 V OV = 54.6 ± 1.09 V T_sc (RST) = 45.3us T_sc (STP) = 48us - RST attempts to reopen GATE after SC detected - STP powers off GATE and requires hard restart"
