File: PresToe_BMS_48V.kicad_sch (KiCad schematic)
At the start: 46 parts, among them J1 XT90PB-F, J2 XT90PB-F, J3 XT30PW-M, J4 S3B-XH-A, J5 S3B-XH-A, J6 Conn_01x06_Pin, Q1 IAUS200N08S5N023ATMA1, Q2 IAUS200N08S5N023ATMA1, Q3 IAUS200N08S5N023ATMA1, SW1 DS04-254-1-01BK-SMT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

Commit message: Basic footprint layout added
Parts:
- removed J5: S3B-XH-A, S3B_XH_A:JST_S3B-XH-A, symbol jst_3pin:S3B-XH-A
- C1, C2, C3: footprint (none) -> Capacitor_SMD:C_0603_1608Metric
- C4: renamed from C_TMR1; footprint (none) -> Capacitor_SMD:C_0603_1608Metric
- C5: renamed from C_BST1; footprint (none) -> Capacitor_SMD:C_0603_1608Metric
- R1, R10, R11, R2, R3, R4, R5, R6, R7, R8, R9, R_FBB1, R_FBT1: footprint (none) -> Resistor_SMD:R_0603_1608Metric
- R12: value 330k -> 51k; footprint (none) -> Resistor_SMD:R_0603_1608Metric
- R13: value 21.5k -> 5k; footprint (none) -> Resistor_SMD:R_0603_1608Metric
- R14: renamed from R_TMR1; footprint (none) -> Resistor_SMD:R_0603_1608Metric
- R15: renamed from R_ISCP1; footprint (none) -> Resistor_SMD:R_0603_1608Metric
- R_SNS1, R_SNS2: footprint (none) -> Resistor_SMD:Custom_R_300u
- U5: footprint SOIC8-N_MC_MCH -> MCP3202:SOIC8-N_MC_MCH
- renumbered D4 to D1, D3 to D2, D2 to D3, J6 to J5, R_VAR1 to P1
Other:
- moved on the sheet: J5

Commit message: finalized, remaining final checks
Parts:
- added H1, H2, H3, H4: MountingHole, MountingHole:MountingHole_3.2mm_M3_Pad_Via, symbol Mechanical:MountingHole
Connections:
- net V_ADC is gone; now on an unnamed net: U4.4 (-IN)
Other:
- note added: "Mounting Holes"

Commit message: fixed bugs, finalized design
Parts:
- removed H3: MountingHole, MountingHole:MountingHole_3.2mm_M3_Pad_Via, symbol Mechanical:MountingHole
- added C10, C11, C6, C7, C8, C9: 0.1uF, Capacitor_SMD:C_0603_1608Metric, symbol Device:C
- added NT1: NetTie_2, NetTie:NetTie-2_SMD_Pad2.0mm, symbol Device:NetTie_2
- P1: footprint 20k_potentiometer:POT_T93YA_VIS -> 89PR20KLF:RES3_89P_TTE
- renumbered H4 to H3
Connections:
- net 5V: now also C10.1, C7.2, C8.2, C9.1
- net GND: now also C10.2, C11.1, C6.2, C7.1, C8.1, C9.2, NT1.2; no longer J1.1, J2.1
- net SPI_VIN: now also C11.2
- net V_in: now also C6.1
- net at U6.11 (IND): now also U5.6 (DOUT); no longer U5.5 (DIN)
- net at U6.14 (OUTA): now also U5.5 (DIN); no longer U5.6 (DOUT)
- new net PWR_GND: J1.1, J2.1, NT1.1
Other:
- moved on the sheet: H3

Commit message: Finalized V1
Parts:
- C2: footprint Capacitor_SMD:C_0603_1608Metric -> Capacitor_SMD:C_0805_2012Metric
- C3: footprint Capacitor_SMD:C_0603_1608Metric -> Capacitor_SMD:C_1210_3225Metric
Changed lines of the file:
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@@
 			)
 		)
-		(property "Footprint" "Capacitor_SMD:C_0603_1608Metric"
+		(property "Footprint" "Capacitor_SMD:C_1210_3225Metric"
 			(at 266.3952 48.26 0)
 			(effects
@@
 			)
 		)
-		(property "Footprint" "Capacitor_SMD:C_0603_1608Metric"
+		(property "Footprint" "Capacitor_SMD:C_0805_2012Metric"
 			(at 196.5452 45.72 0)
 			(effects
